File: schematic/mk2/right_side.sch (KiCad schematic (older format))
At the start: 102 parts

Commit message: schematic: Move the wires for the rows a bit to the right to make them look visually separated from the wires for the columns
Connections:
- wire segments 119 -> 213

Commit message: schematic: Remove the bottom row from the right side and center the components a bit
Parts:
- removed D? (x7): D, symbol D
- removed SW? (x7): SW_PUSH, symbol SW_PUSH
- added D? (x49): D, symbol D
- added SW? (x49): SW_PUSH, symbol SW_PUSH
Connections:
- wire segments 213 -> 372
