File: schematic/mk2/right_side.sch (KiCad schematic (older format))
At the start: 186 parts

Commit message: schematic: KiCad decided to optimise the wires I think
Connections:
- wire segments 372 -> 207

Commit message: schematic: Update to KiCad 5
Parts:
- C?: symbol C -> mylib_experimental:C
- D? (x91): symbol D -> mylib_experimental:D
- R? (x2): symbol R -> mylib_experimental:R
- SW? (x91): symbol SW_PUSH -> mylib_experimental:SW_PUSH
- U?: symbol MCP23017 -> mylib_experimental:MCP23017
Connections:
- wire segments 207 -> 372

Commit message: schematic: Try to make the schematic look like the real hardware
* Delete switches which aren't present.
* Label rows/columns.
* Add connectors for the right side between the rows/columns and the mcp
  board.
* Move the matrix down bit in the left side sheet.
Parts:
- removed D? (x4): D, symbol mylib_experimental:D
- removed SW? (x4): SW_PUSH, symbol mylib_experimental:SW_PUSH
- added J? (x2): Rows, symbol mylib_experimental:Conn_01x06
- added J? (x2): Columns, symbol mylib_experimental:CONN_01X07
Connections:
- net labels added: Col10, Col11, Col12, Col13, Col14, Col8, Col9, Row1, Row2, Row3, Row4, Row5, Row6
- wire segments 372 -> 353

Commit message: schematic: Remove copy pasted left matrix from the right side sheet
Parts:
- removed D? (x49): D, symbol mylib_experimental:D
- removed SW? (x49): SW_PUSH, symbol mylib_experimental:SW_PUSH
Connections:
- wire segments 353 -> 171
