File: schematic/mk2/left_side.sch (KiCad schematic (older format))
At the start: 6 parts

Commit message: schematic: Add switches and diodes to the left side
Parts:
- removed J?: CONN_01X07, symbol CONN_01X07
- added D? (x42): D, symbol D
- added J? (x2): Inputs, symbol Conn_01x06
- added J?: Display, symbol CONN_01X07
- added J? (x2): Outputs, symbol CONN_01X07
- added SW? (x42): SW_PUSH, symbol SW_PUSH
- J?: value CONN_01X07 -> Display
Connections:
- wire segments 81 -> 205
Other:
- moved on the sheet: ARD?, C?, J?, U?
