File: schematic/mk2/left_side.sch (KiCad schematic (older format))
At the start: 94 parts

Commit message: schematic: Update to KiCad 5
Parts:
- ARD?: symbol Arduino_Micro_Socket -> mylib_experimental:Arduino_Micro_Socket
- C?: symbol C -> mylib_experimental:C
- D? (x42): symbol D -> mylib_experimental:D
- J? (x4): symbol CONN_01X07 -> mylib_experimental:CONN_01X07
- J? (x2): symbol Conn_01x06 -> mylib_experimental:Conn_01x06
- SW? (x42): symbol SW_PUSH -> mylib_experimental:SW_PUSH
- U?: symbol 74HC4050 -> mylib_experimental:74HC4050
- U?: symbol TFT128x64 -> mylib_experimental:TFT128x64
Connections:
- wire segments 205 -> 281

Commit message: schematic: Try to make the schematic look like the real hardware
* Delete switches which aren't present.
* Label rows/columns.
* Add connectors for the right side between the rows/columns and the mcp
  board.
* Move the matrix down bit in the left side sheet.
Parts:
- removed D? (x4): D, symbol mylib_experimental:D
- removed SW? (x4): SW_PUSH, symbol mylib_experimental:SW_PUSH
- J? (x2): value Inputs -> Rows
- J? (x2): value Outputs -> Columns
Connections:
- net labels added: Col1, Col2, Col3, Col4, Col5, Col6, Col7, Row1, Row2, Row3, Row4, Row5, Row6
- wire segments 281 -> 269
Other:
- moved on the sheet: J?
