File: schematic/mk1/mcp23017_side_partial/schematic.sch (KiCad schematic (older format))
At the start: 46 parts

Commit message: schematic: Update to KiCad 5
Parts:
- D? (x21): symbol D -> schematic-rescue:D
- P?: symbol CONN_01X04 -> schematic-rescue:CONN_01X04
- R1, R2: symbol R -> schematic-rescue:R
- SW? (x21): symbol SW_PUSH -> schematic-rescue:SW_PUSH
- U?: symbol MCP23017-RESCUE-schematic -> schematic-rescue:MCP23017-RESCUE-schematic
Connections:
- wire segments 71 -> 118
